File: gpsdo.kicad_pcb (KiCad board)
At the start: 2 copper layers, 202 parts, among them J1 OLED, J10 10MHZ_OUT, J11 100MHZ_OUT, J12 10MHZ_OUT, J13 10MHZ_OUT, J14 10MHZ_OUT, J15 10MHZ_OUT, J16 LED, J17 TIMEPULSE, J18 TAP_GPS_TX, J19 TAP_GPS_RX, J2 ARDUINO_UART, J20 TAP_DAC_SDA, J21 TAP_DAC_SCL, J22 TAP_GPS_RF_IN, J23 TAP_GPS_TPLS, J24 TAP_GPS_V_ANT, J3 VOLTMETER, J4 ARDUINO_EXTRA_PINS, J5 POWER_IN, J6 GPS_ANT, J7 10MHZ_OUT, J8 10MHZ_OUT, J9 10MHZ_OUT, U1 TPS79301-EP, U10 MSA-0385, U11 MSA-0385, U12 MSA-0385, U13 MSA-0385, U14 MSA-0385, U15 MSA-0385, U16 MSA-0385, U17 MSA-0385, U18 MSA-0385, U19 MSA-0385, U2 TPS79301-EP, U20 MSA-0385, U21 TPS7A4501DCQT, U3 TPS7A4501DCQT, U4 SN74HC541DWR, U5 DAC8571IDGKR, U6 LEA-M8F, U7 CVSS-945, U8 SN74HC541DWR, U9 MC12080

Commit message: placement_almost_done
Parts:
- moved H2 200.6 mm to (17.8, 152.4)
- moved H1 171.1 mm to (20.3, 17.8)
- moved J5 170.2 mm to (58.9, 150.9), turned to 270 degrees
- moved R11 151.7 mm to (77.5, 41.9), turned to 180 degrees
- moved R20 151.7 mm to (78.5, 72.9)
- moved R2 149.2 mm to (67.6, 25.7)
- moved R12 149.1 mm to (81.5, 41.9), turned to 180 degrees
- moved C76 148.2 mm to (30.5, 47.2), turned to 270 degrees
- moved R10 146.5 mm to (59.2, 51.8), turned to 270 degrees
- moved H4 145.9 mm to (94.0, 152.4)
- moved R8 145.1 mm to (62.7, 50.8), turned to 180 degrees
- moved R50 144.6 mm to (48.3, 132.1)
- moved R47 142.3 mm to (67.6, 136.7), turned to 180 degrees
- moved L2 141.2 mm to (38.1, 18.8), turned to 270 degrees
- moved C79 140.7 mm to (52.1, 133.3), turned to 270 degrees
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Routing:
- net GPS_RF_IN: track 0.00 -> 26.6 mm
- net GPS_ANTENNA: track 0.00 -> 22.9 mm
- net GND: track 0.00 -> 2.80 mm
Other:
- board outline added: 88.9 x 144.8 mm

Commit message: changed_schematic
Parts:
- added J19: USB_DP, Connector_PinHeader_2.54mm:PinHeader_1x01_P2.54mm_Vertical, F.Cu at (42.7, 2.54)
- added J20: SDA, Connector_PinHeader_2.54mm:PinHeader_1x01_P2.54mm_Vertical, F.Cu at (42.7, 7.19)
- added J21: SCL, Connector_PinHeader_2.54mm:PinHeader_1x01_P2.54mm_Vertical, F.Cu at (47.3, 2.54)
- added J22: FREQ0, Connector_PinHeader_2.54mm:PinHeader_1x01_P2.54mm_Vertical, F.Cu at (47.3, 7.19)
- added J23: Freq Out, Connector_PinHeader_2.54mm:PinHeader_1x01_P2.54mm_Vertical, F.Cu at (52.0, 2.54)
- added J24: BOOT, Connector_PinHeader_2.54mm:PinHeader_1x01_P2.54mm_Vertical, F.Cu at (52.0, 7.19)
- added J25: RESET, Connector_PinHeader_2.54mm:PinHeader_1x01_P2.54mm_Vertical, F.Cu at (56.6, 2.54)
- added J26: D_SEL, Connector_PinHeader_2.54mm:PinHeader_1x01_P2.54mm_Vertical, F.Cu at (56.6, 7.19)
- J18: value TAP_GPS_TX -> USB_DM
Connections:
- C2 pad 2: V_IN -> V_MMIC
- C3 pad 2: V_IN -> V_MMIC
- J18 pad 1: GPS_TX -> Net-(J18-Pad1)
- U1 pad 1: V_IN -> V_MMIC
- U1 pad 3: V_IN -> V_MMIC
- U2 pad 1: V_IN -> V_MMIC
- U2 pad 3: V_IN -> V_MMIC
- U6 pad 25: Net-(U6-Pad25) -> Net-(J18-Pad1)

Commit message: temp
Routing:
- net Net-(C49-Pad1): track 0.00 -> 7.32 mm
- net Net-(C48-Pad1): track 0.00 -> 6.71 mm
- net Net-(C61-Pad1): track 0.00 -> 6.46 mm
- net Net-(C60-Pad1): track 0.00 -> 6.46 mm
- net Net-(C46-Pad1): track 0.00 -> 6.46 mm
- net Net-(C59-Pad1): track 0.00 -> 6.46 mm
- net /A6_OUT: track 0.00 -> 6.33 mm
- net /A5_OUT: track 0.00 -> 6.33 mm
- net /A4_OUT: track 0.00 -> 6.33 mm
- net /A1_OUT: track 0.00 -> 6.33 mm
- net /A7_OUT: track 0.00 -> 5.82 mm
- net V_MMIC2: track 0.00 -> 5.45 mm
- net Net-(L11-Pad1): track 0.00 -> 4.30 mm
- net Net-(C62-Pad1): track 0.00 -> 3.66 mm
- net /A2_IN: track 0.00 -> 3.56 mm
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Changed lines of the file:
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@@
     (thickness 1.6)
     (drawings 4)
-    (tracks 17)
+    (tracks 65)
     (zones 0)
     (modules 210)
@@
   (segment (start 33.913 42.795) (end 33.782 42.926) (width 0.7) (layer F.Cu) (net 20))
   (segment (start 33.913 40.223) (end 33.913 42.795) (width 0.7) (layer F.Cu) (net 20))
+  (segment (start 26.1405 80.01) (end 19.812 80.01) (width 1) (layer F.Cu) (net 23))
+  (segment (start 26.1405 120.65) (end 19.812 120.65) (width 1) (layer F.Cu) (net 25))
+  (segment (start 25.8865 140.97) (end 20.066 140.97) (width 1) (layer F.Cu) (net 26))
+  (segment (start 26.1405 90.17) (end 19.812 90.17) (width 1) (layer F.Cu) (net 29))
+  (segment (start 26.1405 110.49) (end 19.812 110.49) (width 1) (layer F.Cu) (net 30))
+  (segment (start 31.0095 134.62) (end 31.242 134.8525) (width 1) (layer F.Cu) (net 35))
+  (segment (start 28.178 134.62) (end 31.0095 134.62) (width 1) (layer F.Cu) (net 35))
+  (segment (start 31.623 80.01) (end 28.2155 80.01) (width 1) (layer F.Cu) (net 46))
+  (segment (start 28.203 79.9975) (end 28.2155 80.01) (width 1) (layer F.Cu) (net 46))
+  (segment (start 28.203 76.962) (end 28.203 79.9975) (width 1) (layer F.Cu) (net 46))
+  (segment (start 26.178 76.937) (end 26.153 76.962) (width 1) (layer F.Cu) (net 47))
+  (segment (start 26.178 73.66) (end 26.178 76.937) (width 1) (layer F.Cu) (net 47))
+  (segment (start 31.623 120.65) (end 28.2155 120.65) (width 1) (layer F.Cu) (net 50))
+  (segment (start 28.203 120.6375) (end 28.2155 120.65) (width 1) (layer F.Cu) (net 50))
+  (segment (start 28.203 117.348) (end 28.203 120.6375) (width 1) (layer F.Cu) (net 50))
+  (segment (start 26.178 113.792) (end 26.178 118.094) (width 1) (layer F.Cu) (net 51))
+  (segment (start 31.623 140.97) (end 27.9615 140.97) (width 1) (layer F.Cu) (net 52))
+  (segment (start 28.203 140.7285) (end 27.9615 140.97) (width 1) (layer F.Cu) (net 52))
+  (segment (start 28.203 137.414) (end 28.203 140.7285) (width 1) (layer F.Cu) (net 52))
+  (segment (start 26.153 134.645) (end 26.178 134.62) (width 1) (layer F.Cu) (net 53))
+  (segment (start 26.153 137.414) (end 26.153 134.645) (width 1) (layer F.Cu) (net 53))
+  (segment (start 31.623 69.85) (end 28.2155 69.85) (width 1) (layer F.Cu) (net 62))
+  (segment (start 28.203 69.8375) (end 28.2155 69.85) (width 1) (layer F.Cu) (net 62))
+  (segment (start 28.203 66.802) (end 28.203 69.8375) (width 1) (layer F.Cu) (net 62))
+  (segment (start 26.153 63.525) (end 26.178 63.5) (width 1) (layer F.Cu) (net 63))
+  (segment (start 26.153 66.802) (end 26.153 63.525) (width 1) (layer F.Cu) (net 63))
+  (segment (start 31.623 90.17) (end 28.2155 90.17) (width 1) (layer F.Cu) (net 64))
+  (segment (start 28.203 90.1575) (end 28.2155 90.17) (width 1) (layer F.Cu) (net 64))
+  (segment (start 28.203 87.122) (end 28.203 90.1575) (width 1) (layer F.Cu) (net 64))
+  (segment (start 26.178 87.097) (end 26.153 87.122) (width 1) (layer F.Cu) (net 65))
+  (segment (start 26.178 84.074) (end 26.178 87.097) (width 1) (layer F.Cu) (net 65))
+  (segment (start 31.623 110.49) (end 28.2155 110.49) (width 1) (layer F.Cu) (net 66))
+  (segment (start 28.203 110.4775) (end 28.2155 110.49) (width 1) (layer F.Cu) (net 66))
+  (segment (start 28.203 107.442) (end 28.203 110.4775) (width 1) (layer F.Cu) (net 66))
+  (segment (start 26.178 107.417) (end 26.153 107.442) (width 1) (layer F.Cu) (net 67))
+  (segment (start 26.178 104.648) (end 26.178 107.417) (width 1) (layer F.Cu) (net 67))
+  (segment (start 31.623 130.81) (end 27.9615 130.81) (width 1) (layer F.Cu) (net 68))
   (segment (start 42.672 43.18) (end 42.113 42.621) (width 0.7) (layer F.Cu) (net 75))
   (segment (start 51.816 43.18) (end 42.672 43.18) (width 0.7) (layer F.Cu) (net 75))
@@
   (segment (start 42.113 42.621) (end 42.113 40.223) (width 0.7) (layer F.Cu) (net 75))
   (segment (start 59.104 33.147) (end 57.023 33.147) (width 0.7) (layer F.Cu) (net 75))
+  (segment (start 36.957 80.01) (end 40.1105 80.01) (width 1) (layer F.Cu) (net 89))
+  (segment (start 36.957 69.85) (end 40.1105 69.85) (width 1) (layer F.Cu) (net 96))
+  (segment (start 42.1855 83.5605) (end 42.18 83.566) (width 1) (layer F.Cu) (net 101))
+  (segment (start 42.1855 80.01) (end 42.1855 83.5605) (width 1) (layer F.Cu) (net 101))
+  (segment (start 42.1855 73.4005) (end 42.18 73.406) (width 1) (layer F.Cu) (net 105))
+  (segment (start 42.1855 69.85) (end 42.1855 73.4005) (width 1) (layer F.Cu) (net 105))
+  (segment (start 30.7125 63.5) (end 30.734 63.4785) (width 1) (layer F.Cu) (net 118))
+  (segment (start 28.178 63.5) (end 30.7125 63.5) (width 1) (layer F.Cu) (net 118))
+  (segment (start 28.178 84.074) (end 28.956 84.074) (width 1) (layer F.Cu) (net 118))
+  (segment (start 29.7395 84.8575) (end 30.734 84.8575) (width 1) (layer F.Cu) (net 118))
+  (segment (start 28.956 84.074) (end 29.7395 84.8575) (width 1) (layer F.Cu) (net 118))
 )

Commit message: Updated footprints
Parts:
- removed the J19 at (53.2, 63.2)
- removed the J20 at (48.6, 67.8)
- removed the J21 at (53.2, 67.8)
- removed the J22 at (57.9, 63.2)
- removed the J23 at (48.6, 72.5)
- removed the J24 at (53.2, 72.5)
- added J27: VCC_OUT, yo6ssw:Single_SMD_Pad, F.Cu at (46.7, 61.6)
- added J28: VDD_USB, yo6ssw:Single_SMD_Pad, F.Cu at (53.3, 61.6)
- added J29: V_ANT, yo6ssw:Single_SMD_Pad, F.Cu at (59.8, 61.6)
- C13, C19, C20: footprint Capacitor_SMD:C_0805_2012Metric_Pad1.18x1.45mm_HandSolder -> yo6ssw:leaded_elec
- C18: value 22uF -> 47uF; footprint Capacitor_SMD:C_0805_2012Metric_Pad1.18x1.45mm_HandSolder -> yo6ssw:leaded_elec
- C78: value 10uF/16V,ESR<3 -> NF
- J18, J19, J20, J21, J22: footprint Connector_PinHeader_2.54mm:PinHeader_1x01_P2.54mm_Vertical -> yo6ssw:Single_SMD_Pad
- J23: renamed from J24; footprint Connector_PinHeader_2.54mm:PinHeader_1x01_P2.54mm_Vertical -> yo6ssw:Single_SMD_Pad
- J24: renamed from J25; footprint Connector_PinHeader_2.54mm:PinHeader_1x01_P2.54mm_Vertical -> yo6ssw:Single_SMD_Pad
- J25: renamed from J26; footprint Connector_PinHeader_2.54mm:PinHeader_1x01_P2.54mm_Vertical -> yo6ssw:Single_SMD_Pad
- J26: renamed from J23; footprint Connector_PinHeader_2.54mm:PinHeader_1x01_P2.54mm_Vertical -> yo6ssw:Single_SMD_Pad
- moved C19 3.30 mm to (97.5, 48.5)
Connections:
- net GPS_V_ANT renamed Net-(J29-Pad1)
- A1 pad 15: Net-(A1-Pad15) -> (no net)
- A1 pad 17: Net-(A1-Pad17) -> (no net)
- A1 pad 18: Net-(A1-Pad18) -> (no net)
- A1 pad 19: Net-(A1-Pad19) -> (no net)
- A1 pad 20: Net-(A1-Pad20) -> (no net)
- A1 pad 21: Net-(A1-Pad21) -> (no net)
- A1 pad 22: Net-(A1-Pad22) -> (no net)
- A1 pad 25: Net-(A1-Pad25) -> (no net)
- A1 pad 26: Net-(A1-Pad26) -> (no net)
- A1 pad 28: Net-(A1-Pad28) -> (no net)
- A1 pad 3: Net-(A1-Pad3) -> (no net)
- C5 pad 2: V_MMIC -> V_MMIC2
- L1 pad 1: V_MMIC -> V_MMIC2
- R47 pad 2: V_ARDUINO -> ARDUINO_5V
- U4 pad 11: Net-(U4-Pad11) -> (no net)
- U4 pad 12: Net-(U4-Pad12) -> (no net)
- U4 pad 13: Net-(U4-Pad13) -> (no net)
- U4 pad 14: Net-(U4-Pad14) -> (no net)
- U4 pad 6: Net-(U4-Pad6) -> (no net)
- U4 pad 7: Net-(U4-Pad7) -> (no net)
- U4 pad 8: Net-(U4-Pad8) -> (no net)
- U4 pad 9: Net-(U4-Pad9) -> (no net)
- U6 pad 20: Net-(U6-Pad20) -> (no net)
- U8 pad 11: Net-(U8-Pad11) -> (no net)
- U8 pad 12: Net-(U8-Pad12) -> (no net)
- U8 pad 13: Net-(U8-Pad13) -> (no net)
- U8 pad 14: Net-(U8-Pad14) -> (no net)
- U8 pad 6: Net-(U8-Pad6) -> (no net)
- U8 pad 7: Net-(U8-Pad7) -> (no net)
- U8 pad 8: Net-(U8-Pad8) -> (no net)
- U8 pad 9: Net-(U8-Pad9) -> (no net)

Commit message: progress
Parts:
- removed J20: SDA, yo6ssw:Single_SMD_Pad
- U6: footprint yo6ssw:LEA-8MF -> RF_GPS:ublox_LEA
- moved C13 43.5 mm to (93.0, 63.8), turned to 0 degrees
- moved J27 41.6 mm to (41.9, 20.3)
- moved J19 40.5 mm to (47.8, 42.7)
- moved J22 35.6 mm to (49.8, 42.7)
- moved J29 29.7 mm to (37.1, 42.4)
- moved J24 25.9 mm to (38.1, 20.6)
- moved C4 23.7 mm to (53.3, 133.3), turned to 90 degrees
- moved J26 22.0 mm to (40.1, 21.1)
- moved C78 21.3 mm to (62.5, 133.3), turned to 90 degrees
- moved J23 20.6 mm to (32.8, 14.7)
- moved J28 20.6 mm to (45.2, 42.7)
- moved J18 18.9 mm to (46.5, 44.5)
- moved J21 18.1 mm to (48.5, 20.6)
- moved J25 17.6 mm to (45.2, 20.6)
- moved J16 13.5 mm to (87.1, 148.3), turned to 270 degrees
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Connections:
- A1 pad 15: (no net) -> Net-(A1-Pad15)
- A1 pad 17: (no net) -> Net-(A1-Pad17)
- A1 pad 18: (no net) -> Net-(A1-Pad18)
- A1 pad 19: (no net) -> Net-(A1-Pad19)
- A1 pad 20: (no net) -> Net-(A1-Pad20)
- A1 pad 21: (no net) -> Net-(A1-Pad21)
- A1 pad 22: (no net) -> Net-(A1-Pad22)
- A1 pad 25: (no net) -> Net-(A1-Pad25)
- A1 pad 26: (no net) -> Net-(A1-Pad26)
- A1 pad 28: (no net) -> Net-(A1-Pad28)
- A1 pad 3: (no net) -> Net-(A1-Pad3)
- C18 pad 1: GND -> Net-(C18-Pad1)
- C18 pad 2: Net-(C18-Pad2) -> GND
- C19 pad 1: GND -> Net-(C19-Pad1)
- C19 pad 2: Net-(C19-Pad2) -> GND
- C20 pad 1: GND -> Net-(C20-Pad1)
- C20 pad 2: Net-(C20-Pad2) -> GND
- C76 pad 2: V_MMIC2 -> V_MMIC
- R11 pad 1: Net-(C18-Pad2) -> Net-(C18-Pad1)
- R12 pad 2: Net-(C18-Pad2) -> Net-(C18-Pad1)
- R13 pad 1: Net-(C19-Pad2) -> Net-(C19-Pad1)
- R14 pad 1: Net-(C20-Pad2) -> Net-(C20-Pad1)
- R14 pad 2: Net-(C19-Pad2) -> Net-(C19-Pad1)
- U21 pad 6: (no net) -> GND
- U3 pad 6: (no net) -> GND
- U4 pad 11: (no net) -> Net-(U4-Pad11)
- U4 pad 12: (no net) -> Net-(U4-Pad12)
- U4 pad 13: (no net) -> Net-(U4-Pad13)
- U4 pad 14: (no net) -> Net-(U4-Pad14)
- U4 pad 6: (no net) -> Net-(U4-Pad6)
- U4 pad 7: (no net) -> Net-(U4-Pad7)
- U4 pad 8: (no net) -> Net-(U4-Pad8)
- U4 pad 9: (no net) -> Net-(U4-Pad9)
- U5 pad 1: Net-(C18-Pad2) -> Net-(C18-Pad1)
- U5 pad 2: Net-(C18-Pad2) -> Net-(C18-Pad1)
- U6 pad 20: (no net) -> Net-(U6-Pad20)
- U7 pad 1: Net-(C20-Pad2) -> Net-(C20-Pad1)
- U8 pad 11: (no net) -> Net-(U8-Pad11)
- U8 pad 12: (no net) -> Net-(U8-Pad12)
- U8 pad 13: (no net) -> Net-(U8-Pad13)
- U8 pad 14: (no net) -> Net-(U8-Pad14)
- U8 pad 6: (no net) -> Net-(U8-Pad6)
- U8 pad 7: (no net) -> Net-(U8-Pad7)
- U8 pad 8: (no net) -> Net-(U8-Pad8)
- U8 pad 9: (no net) -> Net-(U8-Pad9)
Routing:
- net V_MMIC2: track 5.45 -> 248.4 mm
- net GND: track 2.80 -> 231.4 mm, vias 0 -> 29
- net V_MMIC: track 3.16 -> 151.1 mm
- net V_VCXO: track 0.00 -> 114.4 mm
- net V_IN: track 0.00 -> 56.1 mm
- net Net-(C13-Pad1): track 0.00 -> 31.8 mm
- net DAC_SCL: track 0.00 -> 30.1 mm
- net DAC_SDA: track 0.00 -> 29.7 mm
- net Net-(C21-Pad2): track 0.00 -> 24.8 mm
- net Net-(R32-Pad1): track 0.00 -> 22.7 mm
- net Net-(C19-Pad1): track 0.00 -> 21.8 mm
- net Net-(C18-Pad1): track 0.00 -> 20.9 mm
- net VOLTMETER: track 0.00 -> 18.6 mm
- net 10MHZ: track 0.00 -> 17.9 mm
- net Net-(C17-Pad2): track 0.00 -> 15.8 mm
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- added copper zone on B.Cu, net GND

Commit message: progress
Parts:
- moved C1 9.66 mm to (70.6, 20.1), turned to 180 degrees
- moved R3 3.05 mm to (73.2, 36.1)
- moved R4 3.05 mm to (70.9, 36.1)
- moved R2 3.05 mm to (67.6, 22.6)
- moved R1 3.05 mm to (72.6, 32.3)
- moved U4 3.05 mm to (63.8, 30.7)
- moved C11 2.79 mm to (57.7, 38.6)
- moved R11 2.29 mm to (77.5, 44.2)
- moved J17 2.18 mm to (61.2, 18.8)
- moved U7 2.03 mm to (76.5, 45.0)
- moved R12 1.93 mm to (79.8, 41.1)
Routing:
- net V_GPS: track 12.5 -> 101.1 mm
- net GPS_TPLS: track 14.9 -> 42.6 mm
- net V_MMIC: track 151.1 -> 176.0 mm
- net GPS_TX: track 11.6 -> 34.1 mm, vias 0 -> 2
- net GPS_RX: track 12.7 -> 35.0 mm, vias 0 -> 2
- net GPS_RF_IN: track 17.3 -> 36.1 mm, vias 0 -> 2
- net TIMEPULSE: track 0.00 -> 14.0 mm, vias 0 -> 1
- net DAC_SDA: track 29.7 -> 43.4 mm
- net DAC_SCL: track 30.1 -> 42.3 mm
- net Net-(C1-Pad2): track 7.07 -> 14.7 mm
- net GND: track 231.4 -> 229.2 mm, vias 29 -> 48
- net V_VCXO: track 114.4 -> 113.5 mm
- added copper zone on F.Cu, net GND

Commit message: progress
Parts:
- moved R3 11.8 mm to (78.7, 25.7), turned to 0 degrees
- moved C1 8.68 mm to (78.7, 23.1)
- moved R14 8.44 mm to (85.3, 43.2), turned to 0 degrees
- moved C21 8.33 mm to (72.1, 72.4)
- moved R2 7.55 mm to (72.6, 28.2), turned to 90 degrees
- moved C18 3.05 mm to (91.9, 39.6)
- moved R13 2.34 mm to (85.1, 39.6), turned to 90 degrees
- moved C13 2.03 mm to (90.9, 63.8)
- moved C20 1.78 mm to (91.9, 55.4)
- moved C19 1.61 mm to (92.2, 47.8)
Routing:
- net Net-(D4-Pad1): track 0.00 -> 208.3 mm, vias 0 -> 4
- net A2G_TX: track 0.00 -> 180.5 mm
- net 10MHZ: track 17.9 -> 94.9 mm, vias 0 -> 2
- net ARDUINO_5V: track 8.16 -> 74.6 mm
- net Net-(C19-Pad1): track 21.8 -> 0.00 mm
- net Net-(C20-Pad1): track 14.4 -> 0.00 mm
- net ARDUINO_UART_RX: track 0.00 -> 14.0 mm
- net Net-(R3-Pad1): track 4.79 -> 15.9 mm
- net ARDUINO_UART_TX: track 0.00 -> 9.22 mm
- net (no net): track 0.00 -> 4.17 mm, vias 0 -> 1
- net GND: track 229.2 -> 232.3 mm
- net Net-(C18-Pad1): track 21.1 -> 18.1 mm

Commit message: final
Parts:
- added REF**: PinHeader_1x01_P2.54mm_Vertical, Connector_PinHeader_2.54mm:PinHeader_1x01_P2.54mm_Vertical, F.Cu at (86.4, 76.2)
- added REF**: PinHeader_1x01_P2.54mm_Vertical, Connector_PinHeader_2.54mm:PinHeader_1x01_P2.54mm_Vertical, F.Cu at (94.0, 78.7)
- added REF**: PinHeader_1x01_P2.54mm_Vertical, Connector_PinHeader_2.54mm:PinHeader_1x01_P2.54mm_Vertical, F.Cu at (96.5, 78.7)
- added REF**: PinHeader_1x01_P2.54mm_Vertical, Connector_PinHeader_2.54mm:PinHeader_1x01_P2.54mm_Vertical, F.Cu at (76.2, 81.3)
- added REF**: PinHeader_1x01_P2.54mm_Vertical, Connector_PinHeader_2.54mm:PinHeader_1x01_P2.54mm_Vertical, F.Cu at (78.7, 81.3)
- added REF**: PinHeader_1x01_P2.54mm_Vertical, Connector_PinHeader_2.54mm:PinHeader_1x01_P2.54mm_Vertical, F.Cu at (81.3, 81.3)
- added REF**: PinHeader_1x01_P2.54mm_Vertical, Connector_PinHeader_2.54mm:PinHeader_1x01_P2.54mm_Vertical, F.Cu at (83.8, 81.3)
- added REF**: PinHeader_1x01_P2.54mm_Vertical, Connector_PinHeader_2.54mm:PinHeader_1x01_P2.54mm_Vertical, F.Cu at (86.4, 81.3)
- added REF**: PinHeader_1x01_P2.54mm_Vertical, Connector_PinHeader_2.54mm:PinHeader_1x01_P2.54mm_Vertical, F.Cu at (88.9, 81.3)
- added REF**: PinHeader_1x01_P2.54mm_Vertical, Connector_PinHeader_2.54mm:PinHeader_1x01_P2.54mm_Vertical, F.Cu at (91.4, 81.3)
- added REF**: PinHeader_1x01_P2.54mm_Vertical, Connector_PinHeader_2.54mm:PinHeader_1x01_P2.54mm_Vertical, F.Cu at (94.0, 81.3)
- added REF**: PinHeader_1x01_P2.54mm_Vertical, Connector_PinHeader_2.54mm:PinHeader_1x01_P2.54mm_Vertical, F.Cu at (88.9, 76.2)
- added REF**: PinHeader_1x01_P2.54mm_Vertical, Connector_PinHeader_2.54mm:PinHeader_1x01_P2.54mm_Vertical, F.Cu at (96.5, 81.3)
- added REF**: PinHeader_1x01_P2.54mm_Vertical, Connector_PinHeader_2.54mm:PinHeader_1x01_P2.54mm_Vertical, F.Cu at (73.7, 83.8)
- added REF**: PinHeader_1x01_P2.54mm_Vertical, Connector_PinHeader_2.54mm:PinHeader_1x01_P2.54mm_Vertical, F.Cu at (76.2, 83.8)
- added REF**: PinHeader_1x01_P2.54mm_Vertical, Connector_PinHeader_2.54mm:PinHeader_1x01_P2.54mm_Vertical, F.Cu at (78.7, 83.8)
- added REF**: PinHeader_1x01_P2.54mm_Vertical, Connector_PinHeader_2.54mm:PinHeader_1x01_P2.54mm_Vertical, F.Cu at (81.3, 83.8)
- added REF**: PinHeader_1x01_P2.54mm_Vertical, Connector_PinHeader_2.54mm:PinHeader_1x01_P2.54mm_Vertical, F.Cu at (83.8, 83.8)
- added REF**: PinHeader_1x01_P2.54mm_Vertical, Connector_PinHeader_2.54mm:PinHeader_1x01_P2.54mm_Vertical, F.Cu at (86.4, 83.8)
- added REF**: PinHeader_1x01_P2.54mm_Vertical, Connector_PinHeader_2.54mm:PinHeader_1x01_P2.54mm_Vertical, F.Cu at (88.9, 83.8)
- added REF**: PinHeader_1x01_P2.54mm_Vertical, Connector_PinHeader_2.54mm:PinHeader_1x01_P2.54mm_Vertical, F.Cu at (91.4, 83.8)
- added REF**: PinHeader_1x01_P2.54mm_Vertical, Connector_PinHeader_2.54mm:PinHeader_1x01_P2.54mm_Vertical, F.Cu at (94.0, 83.8)
- added REF**: PinHeader_1x01_P2.54mm_Vertical, Connector_PinHeader_2.54mm:PinHeader_1x01_P2.54mm_Vertical, F.Cu at (91.4, 76.2)
- added REF**: PinHeader_1x01_P2.54mm_Vertical, Connector_PinHeader_2.54mm:PinHeader_1x01_P2.54mm_Vertical, F.Cu at (96.5, 83.8)
- added REF**: PinHeader_1x01_P2.54mm_Vertical, Connector_PinHeader_2.54mm:PinHeader_1x01_P2.54mm_Vertical, F.Cu at (73.7, 86.4)
- added REF**: PinHeader_1x01_P2.54mm_Vertical, Connector_PinHeader_2.54mm:PinHeader_1x01_P2.54mm_Vertical, F.Cu at (76.2, 86.4)
- added REF**: PinHeader_1x01_P2.54mm_Vertical, Connector_PinHeader_2.54mm:PinHeader_1x01_P2.54mm_Vertical, F.Cu at (78.7, 86.4)
- added REF**: PinHeader_1x01_P2.54mm_Vertical, Connector_PinHeader_2.54mm:PinHeader_1x01_P2.54mm_Vertical, F.Cu at (81.3, 86.4)
- added REF**: PinHeader_1x01_P2.54mm_Vertical, Connector_PinHeader_2.54mm:PinHeader_1x01_P2.54mm_Vertical, F.Cu at (83.8, 86.4)
- added REF**: PinHeader_1x01_P2.54mm_Vertical, Connector_PinHeader_2.54mm:PinHeader_1x01_P2.54mm_Vertical, F.Cu at (86.4, 86.4)
- added REF**: PinHeader_1x01_P2.54mm_Vertical, Connector_PinHeader_2.54mm:PinHeader_1x01_P2.54mm_Vertical, F.Cu at (88.9, 86.4)
- added REF**: PinHeader_1x01_P2.54mm_Vertical, Connector_PinHeader_2.54mm:PinHeader_1x01_P2.54mm_Vertical, F.Cu at (91.4, 86.4)
- added REF**: PinHeader_1x01_P2.54mm_Vertical, Connector_PinHeader_2.54mm:PinHeader_1x01_P2.54mm_Vertical, F.Cu at (94.0, 86.4)
- added REF**: PinHeader_1x01_P2.54mm_Vertical, Connector_PinHeader_2.54mm:PinHeader_1x01_P2.54mm_Vertical, F.Cu at (94.0, 76.2)
- added REF**: PinHeader_1x01_P2.54mm_Vertical, Connector_PinHeader_2.54mm:PinHeader_1x01_P2.54mm_Vertical, F.Cu at (96.5, 86.4)
- added REF**: PinHeader_1x01_P2.54mm_Vertical, Connector_PinHeader_2.54mm:PinHeader_1x01_P2.54mm_Vertical, F.Cu at (73.7, 88.9)
- added REF**: PinHeader_1x01_P2.54mm_Vertical, Connector_PinHeader_2.54mm:PinHeader_1x01_P2.54mm_Vertical, F.Cu at (76.2, 88.9)
- added REF**: PinHeader_1x01_P2.54mm_Vertical, Connector_PinHeader_2.54mm:PinHeader_1x01_P2.54mm_Vertical, F.Cu at (78.7, 88.9)
- added REF**: PinHeader_1x01_P2.54mm_Vertical, Connector_PinHeader_2.54mm:PinHeader_1x01_P2.54mm_Vertical, F.Cu at (81.3, 88.9)
- added REF**: PinHeader_1x01_P2.54mm_Vertical, Connector_PinHeader_2.54mm:PinHeader_1x01_P2.54mm_Vertical, F.Cu at (83.8, 88.9)
- added REF**: PinHeader_1x01_P2.54mm_Vertical, Connector_PinHeader_2.54mm:PinHeader_1x01_P2.54mm_Vertical, F.Cu at (86.4, 88.9)
- added REF**: PinHeader_1x01_P2.54mm_Vertical, Connector_PinHeader_2.54mm:PinHeader_1x01_P2.54mm_Vertical, F.Cu at (88.9, 88.9)
- added REF**: PinHeader_1x01_P2.54mm_Vertical, Connector_PinHeader_2.54mm:PinHeader_1x01_P2.54mm_Vertical, F.Cu at (91.4, 88.9)
- added REF**: PinHeader_1x01_P2.54mm_Vertical, Connector_PinHeader_2.54mm:PinHeader_1x01_P2.54mm_Vertical, F.Cu at (94.0, 88.9)
- added REF**: PinHeader_1x01_P2.54mm_Vertical, Connector_PinHeader_2.54mm:PinHeader_1x01_P2.54mm_Vertical, F.Cu at (96.5, 76.2)
- added REF**: PinHeader_1x01_P2.54mm_Vertical, Connector_PinHeader_2.54mm:PinHeader_1x01_P2.54mm_Vertical, F.Cu at (96.5, 88.9)
- added REF**: PinHeader_1x01_P2.54mm_Vertical, Connector_PinHeader_2.54mm:PinHeader_1x01_P2.54mm_Vertical, F.Cu at (73.7, 91.4)
- added REF**: PinHeader_1x01_P2.54mm_Vertical, Connector_PinHeader_2.54mm:PinHeader_1x01_P2.54mm_Vertical, F.Cu at (76.2, 91.4)
- added REF**: PinHeader_1x01_P2.54mm_Vertical, Connector_PinHeader_2.54mm:PinHeader_1x01_P2.54mm_Vertical, F.Cu at (78.7, 91.4)
- added REF**: PinHeader_1x01_P2.54mm_Vertical, Connector_PinHeader_2.54mm:PinHeader_1x01_P2.54mm_Vertical, F.Cu at (81.3, 91.4)
- added REF**: PinHeader_1x01_P2.54mm_Vertical, Connector_PinHeader_2.54mm:PinHeader_1x01_P2.54mm_Vertical, F.Cu at (83.8, 91.4)
- added REF**: PinHeader_1x01_P2.54mm_Vertical, Connector_PinHeader_2.54mm:PinHeader_1x01_P2.54mm_Vertical, F.Cu at (86.4, 91.4)
- added REF**: PinHeader_1x01_P2.54mm_Vertical, Connector_PinHeader_2.54mm:PinHeader_1x01_P2.54mm_Vertical, F.Cu at (88.9, 91.4)
- added REF**: PinHeader_1x01_P2.54mm_Vertical, Connector_PinHeader_2.54mm:PinHeader_1x01_P2.54mm_Vertical, F.Cu at (91.4, 91.4)
- added REF**: PinHeader_1x01_P2.54mm_Vertical, Connector_PinHeader_2.54mm:PinHeader_1x01_P2.54mm_Vertical, F.Cu at (94.0, 91.4)
- added REF**: PinHeader_1x01_P2.54mm_Vertical, Connector_PinHeader_2.54mm:PinHeader_1x01_P2.54mm_Vertical, F.Cu at (83.8, 78.7)
- added REF**: PinHeader_1x01_P2.54mm_Vertical, Connector_PinHeader_2.54mm:PinHeader_1x01_P2.54mm_Vertical, F.Cu at (96.5, 91.4)
- added REF**: PinHeader_1x01_P2.54mm_Vertical, Connector_PinHeader_2.54mm:PinHeader_1x01_P2.54mm_Vertical, F.Cu at (73.7, 94.0)
- added REF**: PinHeader_1x01_P2.54mm_Vertical, Connector_PinHeader_2.54mm:PinHeader_1x01_P2.54mm_Vertical, F.Cu at (76.2, 94.0)
- added REF**: PinHeader_1x01_P2.54mm_Vertical, Connector_PinHeader_2.54mm:PinHeader_1x01_P2.54mm_Vertical, F.Cu at (78.7, 94.0)
- added REF**: PinHeader_1x01_P2.54mm_Vertical, Connector_PinHeader_2.54mm:PinHeader_1x01_P2.54mm_Vertical, F.Cu at (81.3, 94.0)
- added REF**: PinHeader_1x01_P2.54mm_Vertical, Connector_PinHeader_2.54mm:PinHeader_1x01_P2.54mm_Vertical, F.Cu at (83.8, 94.0)
- added REF**: PinHeader_1x01_P2.54mm_Vertical, Connector_PinHeader_2.54mm:PinHeader_1x01_P2.54mm_Vertical, F.Cu at (86.4, 94.0)
- added REF**: PinHeader_1x01_P2.54mm_Vertical, Connector_PinHeader_2.54mm:PinHeader_1x01_P2.54mm_Vertical, F.Cu at (88.9, 94.0)
- added REF**: PinHeader_1x01_P2.54mm_Vertical, Connector_PinHeader_2.54mm:PinHeader_1x01_P2.54mm_Vertical, F.Cu at (91.4, 94.0)
- added REF**: PinHeader_1x01_P2.54mm_Vertical, Connector_PinHeader_2.54mm:PinHeader_1x01_P2.54mm_Vertical, F.Cu at (94.0, 94.0)
- added REF**: PinHeader_1x01_P2.54mm_Vertical, Connector_PinHeader_2.54mm:PinHeader_1x01_P2.54mm_Vertical, F.Cu at (86.4, 78.7)
- added REF**: PinHeader_1x01_P2.54mm_Vertical, Connector_PinHeader_2.54mm:PinHeader_1x01_P2.54mm_Vertical, F.Cu at (96.5, 94.0)
- added REF**: PinHeader_1x01_P2.54mm_Vertical, Connector_PinHeader_2.54mm:PinHeader_1x01_P2.54mm_Vertical, F.Cu at (73.7, 96.5)
- added REF**: PinHeader_1x01_P2.54mm_Vertical, Connector_PinHeader_2.54mm:PinHeader_1x01_P2.54mm_Vertical, F.Cu at (76.2, 96.5)
- added REF**: PinHeader_1x01_P2.54mm_Vertical, Connector_PinHeader_2.54mm:PinHeader_1x01_P2.54mm_Vertical, F.Cu at (78.7, 96.5)
- added REF**: PinHeader_1x01_P2.54mm_Vertical, Connector_PinHeader_2.54mm:PinHeader_1x01_P2.54mm_Vertical, F.Cu at (81.3, 96.5)
- added REF**: PinHeader_1x01_P2.54mm_Vertical, Connector_PinHeader_2.54mm:PinHeader_1x01_P2.54mm_Vertical, F.Cu at (83.8, 96.5)
- added REF**: PinHeader_1x01_P2.54mm_Vertical, Connector_PinHeader_2.54mm:PinHeader_1x01_P2.54mm_Vertical, F.Cu at (86.4, 96.5)
- added REF**: PinHeader_1x01_P2.54mm_Vertical, Connector_PinHeader_2.54mm:PinHeader_1x01_P2.54mm_Vertical, F.Cu at (88.9, 96.5)
- added REF**: PinHeader_1x01_P2.54mm_Vertical, Connector_PinHeader_2.54mm:PinHeader_1x01_P2.54mm_Vertical, F.Cu at (91.4, 96.5)
- added REF**: PinHeader_1x01_P2.54mm_Vertical, Connector_PinHeader_2.54mm:PinHeader_1x01_P2.54mm_Vertical, F.Cu at (94.0, 96.5)
- added REF**: PinHeader_1x01_P2.54mm_Vertical, Connector_PinHeader_2.54mm:PinHeader_1x01_P2.54mm_Vertical, F.Cu at (88.9, 78.7)
- added REF**: PinHeader_1x01_P2.54mm_Vertical, Connector_PinHeader_2.54mm:PinHeader_1x01_P2.54mm_Vertical, F.Cu at (96.5, 96.5)
- added REF**: PinHeader_1x01_P2.54mm_Vertical, Connector_PinHeader_2.54mm:PinHeader_1x01_P2.54mm_Vertical, F.Cu at (73.7, 99.1)
- added REF**: PinHeader_1x01_P2.54mm_Vertical, Connector_PinHeader_2.54mm:PinHeader_1x01_P2.54mm_Vertical, F.Cu at (76.2, 99.1)
- added REF**: PinHeader_1x01_P2.54mm_Vertical, Connector_PinHeader_2.54mm:PinHeader_1x01_P2.54mm_Vertical, F.Cu at (78.7, 99.1)
- added REF**: PinHeader_1x01_P2.54mm_Vertical, Connector_PinHeader_2.54mm:PinHeader_1x01_P2.54mm_Vertical, F.Cu at (81.3, 99.1)
- added REF**: PinHeader_1x01_P2.54mm_Vertical, Connector_PinHeader_2.54mm:PinHeader_1x01_P2.54mm_Vertical, F.Cu at (83.8, 99.1)
- added REF**: PinHeader_1x01_P2.54mm_Vertical, Connector_PinHeader_2.54mm:PinHeader_1x01_P2.54mm_Vertical, F.Cu at (86.4, 99.1)
- added REF**: PinHeader_1x01_P2.54mm_Vertical, Connector_PinHeader_2.54mm:PinHeader_1x01_P2.54mm_Vertical, F.Cu at (88.9, 99.1)
- added REF**: PinHeader_1x01_P2.54mm_Vertical, Connector_PinHeader_2.54mm:PinHeader_1x01_P2.54mm_Vertical, F.Cu at (91.4, 99.1)
- added REF**: PinHeader_1x01_P2.54mm_Vertical, Connector_PinHeader_2.54mm:PinHeader_1x01_P2.54mm_Vertical, F.Cu at (94.0, 99.1)
- added REF**: PinHeader_1x01_P2.54mm_Vertical, Connector_PinHeader_2.54mm:PinHeader_1x01_P2.54mm_Vertical, F.Cu at (91.4, 78.7)
- added REF**: PinHeader_1x01_P2.54mm_Vertical, Connector_PinHeader_2.54mm:PinHeader_1x01_P2.54mm_Vertical, F.Cu at (96.5, 99.1)
- moved J2 19.1 mm to (67.6, 110.5), turned to 180 degrees
- moved L4 8.32 mm to (74.9, 77.0), turned to 90 degrees
- moved C25 8.13 mm to (73.2, 80.5)
- moved J6 6.60 mm to (20.1, 41.7)
- moved C37 4.31 mm to (62.0, 102.1), turned to 270 degrees
- moved D3 3.34 mm to (24.9, 40.4), turned to 90 degrees
- moved J11 2.29 mm to (19.8, 55.4)
- moved U7 1.02 mm to (76.5, 46.0)
- moved L14 0.51 mm to (47.5, 96.3)
Routing:
- net V_MMIC: track 176.0 -> 342.4 mm
- net GND: track 232.3 -> 276.7 mm, vias 48 -> 61
- net Net-(C20-Pad1): track 0.00 -> 18.2 mm
- net A2G_TX: track 180.5 -> 162.5 mm, vias 0 -> 1
- net ARDUINO_5V: track 74.6 -> 56.8 mm
- net Net-(D4-Pad1): track 208.3 -> 191.6 mm
- net V_VCXO: track 113.5 -> 103.5 mm
- net Net-(C19-Pad1): track 0.00 -> 8.71 mm
- net ARDUINO_UART_RX: track 14.0 -> 7.87 mm
- net GPS_ANTENNA: track 22.0 -> 16.3 mm
- net (no net): track 4.17 -> 0.00 mm
- net V_GPS: track 101.2 -> 97.4 mm
- net 10MHZ: track 94.9 -> 91.2 mm
- net V_MMIC2: track 248.4 -> 250.6 mm, vias 0 -> 2
- net GPS_TPLS: track 42.6 -> 44.7 mm
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- added copper zone on B.Cu, net V_MMIC
- added copper zone on F.Cu, net V_MMIC
Other:
- board text added: "GPS Disciplined Ref 20210115"
