File: gpsdo.kicad_pcb (KiCad board)
At the start: 2 copper layers, 144.8 x 88.9 mm, 296 parts, among them J1 OLED, J10 10MHZ_OUT, J11 100MHZ_OUT, J12 10MHZ_OUT, J13 10MHZ_OUT, J14 10MHZ_OUT, J15 10MHZ_OUT, J16 LED, J17 TIMEPULSE, J18 USB_DM, J19 USB_DP, J2 ARDUINO_UART, J21 SCL, J22 FREQ0, J23 BOOT, J24 RESET, J25 D_SEL, J26 Freq Out, J27 VCC_OUT, J28 VDD_USB, J29 V_ANT, J3 VOLTMETER, J4 ARDUINO_EXTRA_PINS, J5 POWER_IN, J6 GPS_ANT, J7 10MHZ_OUT, J8 10MHZ_OUT, J9 10MHZ_OUT, U1 TPS79301-EP, U10 MSA-0385, U11 MSA-0385, U12 MSA-0385, U13 MSA-0385, U14 MSA-0385, U15 MSA-0385, U16 MSA-0385, U17 MSA-0385, U18 MSA-0385, U19 MSA-0385, U2 TPS79301-EP, U20 MSA-0385, U21 TPS7A4501DCQT, U3 TPS7A4501DCQT, U4 SN74HC541DWR, U5 DAC8571IDGKR, U6 LEA-M8F, U7 CVSS-945, U8 SN74HC541DWR, U9 MC12080

Commit message: moved_track_again
Routing:
- net GND: track 276.7 -> 279.4 mm
- net GPS_TPLS: track 42.5 -> 43.2 mm
Changed lines of the file:
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@@
     (thickness 1.6)
     (drawings 5)
-    (tracks 1065)
+    (tracks 1069)
     (zones 0)
     (modules 296)
@@
   (via (at 77.343 88.773) (size 0.8) (drill 0.4) (layers F.Cu B.Cu) (net 4))
   (via (at 93.345 101.727) (size 0.8) (drill 0.4) (layers F.Cu B.Cu) (net 4))
-  (via (at 88.646 90.932) (size 0.8) (drill 0.4) (layers F.Cu B.Cu) (net 4))
   (segment (start 91.567 117.752) (end 92.352 116.967) (width 0.25) (layer F.Cu) (net 4))
   (segment (start 91.567 119.253) (end 91.567 117.752) (width 0.25) (layer F.Cu) (net 4))
@@
   (segment (start 196.5835 91.059) (end 196.5835 78.2445) (width 2) (layer F.Cu) (net 4))
   (segment (start 196.5835 91.059) (end 196.5835 95.2625) (width 2) (layer F.Cu) (net 4))
+  (via (at 88.646 88.70901) (size 0.8) (drill 0.4) (layers F.Cu B.Cu) (net 4))
+  (segment (start 88.646 91.44) (end 88.646 88.70901) (width 0.6) (layer F.Cu) (net 4))
   (segment (start 187.833 67.691) (end 187.833 70.993) (width 1) (layer B.Cu) (net 5))
   (segment (start 187.833 70.993) (end 189.103 72.263) (width 1) (layer B.Cu) (net 5))
@@
   (segment (start 97.218 88.265) (end 97.155 88.265) (width 1) (layer B.Cu) (net 75))
   (segment (start 94.869 87.757) (end 97.218 88.265) (width 1) (layer B.Cu) (net 75))
-  (segment (start 82.55 83.566) (end 82.55 82.755) (width 0.7) (layer F.Cu) (net 75))
-  (segment (start 86.741 87.757) (end 82.55 83.566) (width 0.7) (layer F.Cu) (net 75))
-  (segment (start 94.869 87.757) (end 86.741 87.757) (width 0.7) (layer F.Cu) (net 75))
+  (segment (start 82.55 83.78) (end 82.55 82.755) (width 0.7) (layer F.Cu) (net 75))
+  (segment (start 85.116989 86.346989) (end 82.55 83.78) (width 0.7) (layer F.Cu) (net 75))
+  (segment (start 89.394989 86.346989) (end 85.116989 86.346989) (width 0.7) (layer F.Cu) (net 75))
+  (segment (start 90.805 87.757) (end 89.394989 86.346989) (width 0.7) (layer F.Cu) (net 75))
+  (segment (start 94.869 87.757) (end 90.805 87.757) (width 0.7) (layer F.Cu) (net 75))
   (segment (start 83.82 69.326) (end 83.709 69.215) (width 0.45) (layer F.Cu) (net 76))
   (segment (start 83.82 73.455) (end 83.82 69.326) (width 0.45) (layer F.Cu) (net 76))
@@
   (segment (start 78.597 66.167) (end 77.5755 66.167) (width 0.65) (layer F.Cu) (net 76))
   (segment (start 92.347 92.211) (end 92.347 92.057) (width 0.45) (layer F.Cu) (net 77))
-  (segment (start 89.036 88.9) (end 92.347 92.211) (width 0.45) (layer F.Cu) (net 77))
-  (segment (start 79.251498 88.9) (end 89.036 88.9) (width 0.45) (layer F.Cu) (net 77))
-  (segment (start 75.870258 85.51876) (end 79.251498 88.9) (width 0.45) (layer F.Cu) (net 77))
-  (segment (start 74.802248 85.51876) (end 75.870258 85.51876) (width 0.45) (layer F.Cu) (net 77))
+  (segment (start 92.347 91.077) (end 92.347 92.211) (width 0.45) (layer F.Cu) (net 77))
+  (segment (start 89.154 87.884) (end 92.347 91.077) (width 0.45) (layer F.Cu) (net 77))
+  (segment (start 78.235498 87.884) (end 89.154 87.884) (width 0.45) (layer F.Cu) (net 77))
+  (segment (start 75.870258 85.51876) (end 78.235498 87.884) (width 0.45) (layer F.Cu) (net 77))
   (segment (start 73.058978 83.77549) (end 74.802248 85.51876) (width 0.45) (layer F.Cu) (net 77))
   (segment (start 73.058978 79.153514) (end 73.058978 83.77549) (width 0.45) (layer F.Cu) (net 77))
-  (segment (start 74.645512 77.56698) (end 73.058978 79.153514) (width 0.45) (layer F.Cu) (net 77))
+  (segment (start 74.802248 85.51876) (end 75.870258 85.51876) (width 0.45) (layer F.Cu) (net 77))
   (segment (start 82.00302 77.56698) (end 74.645512 77.56698) (width 0.45) (layer F.Cu) (net 77))
   (segment (start 85.09 74.48) (end 82.00302 77.56698) (width 0.45) (layer F.Cu) (net 77))
+  (segment (start 74.645512 77.56698) (end 73.058978 79.153514) (width 0.45) (layer F.Cu) (net 77))
   (segment (start 85.09 73.455) (end 85.09 74.48) (width 0.45) (layer F.Cu) (net 77))
   (segment (start 72.443239 94.557001) (end 71.812999 93.926761) (width 0.5) (layer F.Cu) (net 78))

Commit message: GND_plane
Routing:
- net V_MMIC: track 342.4 -> 378.6 mm
- net GND: vias 61 -> 101
- removed copper zone on B.Cu, net V_MMIC
- removed copper zone on F.Cu, net V_MMIC
Changed lines of the file:
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@@
     (thickness 1.6)
     (drawings 5)
-    (tracks 1069)
+    (tracks 1127)
     (zones 0)
     (modules 296)
@@
     (38 B.Mask user hide)
     (39 F.Mask user hide)
-    (40 Dwgs.User user hide)
+    (40 Dwgs.User user)
     (41 Cmts.User user hide)
     (42 Eco1.User user hide)
@@
   (via (at 88.646 88.70901) (size 0.8) (drill 0.4) (layers F.Cu B.Cu) (net 4))
   (segment (start 88.646 91.44) (end 88.646 88.70901) (width 0.6) (layer F.Cu) (net 4))
+  (via (at 66.548 106.68) (size 0.8) (drill 0.4) (layers F.Cu B.Cu) (net 4))
+  (via (at 66.548 61.722) (size 0.8) (drill 0.4) (layers F.Cu B.Cu) (net 4))
+  (via (at 84.582 41.91) (size 0.8) (drill 0.4) (layers F.Cu B.Cu) (net 4))
+  (via (at 84.836 49.022) (size 0.8) (drill 0.4) (layers F.Cu B.Cu) (net 4))
+  (via (at 86.106 65.786) (size 0.8) (drill 0.4) (layers F.Cu B.Cu) (net 4))
+  (via (at 96.266 53.594) (size 0.8) (drill 0.4) (layers F.Cu B.Cu) (net 4))
+  (via (at 99.568 58.928) (size 0.8) (drill 0.4) (layers F.Cu B.Cu) (net 4))
+  (via (at 104.394 59.944) (size 0.8) (drill 0.4) (layers F.Cu B.Cu) (net 4))
+  (via (at 119.888 56.388) (size 0.8) (drill 0.4) (layers F.Cu B.Cu) (net 4))
+  (via (at 121.666 50.546) (size 0.8) (drill 0.4) (layers F.Cu B.Cu) (net 4))
+  (via (at 114.554 78.994) (size 0.8) (drill 0.4) (layers F.Cu B.Cu) (net 4))
+  (via (at 109.474 85.09) (size 0.8) (drill 0.4) (layers F.Cu B.Cu) (net 4))
+  (via (at 120.142 100.33) (size 0.8) (drill 0.4) (layers F.Cu B.Cu) (net 4))
+  (via (at 123.444 97.536) (size 0.8) (drill 0.4) (layers F.Cu B.Cu) (net 4))
+  (via (at 134.874 94.996) (size 0.8) (drill 0.4) (layers F.Cu B.Cu) (net 4))
+  (via (at 146.558 91.186) (size 0.8) (drill 0.4) (layers F.Cu B.Cu) (net 4))
+  (via (at 153.416 82.042) (size 0.8) (drill 0.4) (layers F.Cu B.Cu) (net 4))
+  (via (at 137.414 81.026) (size 0.8) (drill 0.4) (layers F.Cu B.Cu) (net 4))
+  (via (at 144.78 79.756) (size 0.8) (drill 0.4) (layers F.Cu B.Cu) (net 4))
+  (via (at 157.226 76.962) (size 0.8) (drill 0.4) (layers F.Cu B.Cu) (net 4))
+  (via (at 192.532 74.93) (size 0.8) (drill 0.4) (layers F.Cu B.Cu) (net 4))
+  (via (at 171.45 80.01) (size 0.8) (drill 0.4) (layers F.Cu B.Cu) (net 4))
+  (via (at 175.768 83.82) (size 0.8) (drill 0.4) (layers F.Cu B.Cu) (net 4))
+  (via (at 174.498 91.186) (size 0.8) (drill 0.4) (layers F.Cu B.Cu) (net 4))
+  (via (at 182.372 88.9) (size 0.8) (drill 0.4) (layers F.Cu B.Cu) (net 4))
+  (via (at 155.448 50.8) (size 0.8) (drill 0.4) (layers F.Cu B.Cu) (net 4))
+  (via (at 162.56 43.942) (size 0.8) (drill 0.4) (layers F.Cu B.Cu) (net 4))
+  (via (at 163.322 50.038) (size 0.8) (drill 0.4) (layers F.Cu B.Cu) (net 4))
+  (via (at 186.436 43.942) (size 0.8) (drill 0.4) (layers F.Cu B.Cu) (net 4))
+  (via (at 196.596 54.864) (size 0.8) (drill 0.4) (layers F.Cu B.Cu) (net 4))
+  (via (at 189.992 41.91) (size 0.8) (drill 0.4) (layers F.Cu B.Cu) (net 4))
+  (via (at 201.422 72.644) (size 0.8) (drill 0.4) (layers F.Cu B.Cu) (net 4))
+  (via (at 200.66 60.452) (size 0.8) (drill 0.4) (layers F.Cu B.Cu) (net 4))
+  (via (at 206.502 76.454) (size 0.8) (drill 0.4) (layers F.Cu B.Cu) (net 4))
+  (via (at 200.66 77.724) (size 0.8) (drill 0.4) (layers F.Cu B.Cu) (net 4))
+  (via (at 188.468 74.168) (size 0.8) (drill 0.4) (layers F.Cu B.Cu) (net 4))
+  (via (at 164.846 70.612) (size 0.8) (drill 0.4) (layers F.Cu B.Cu) (net 4))
+  (via (at 187.452 97.282) (size 0.8) (drill 0.4) (layers F.Cu B.Cu) (net 4))
+  (via (at 169.672 91.186) (size 0.8) (drill 0.4) (layers F.Cu B.Cu) (net 4))
+  (via (at 155.448 65.278) (size 0.8) (drill 0.4) (layers F.Cu B.Cu) (net 4))
   (segment (start 187.833 67.691) (end 187.833 70.993) (width 1) (layer B.Cu) (net 5))
   (segment (start 187.833 70.993) (end 189.103 72.263) (width 1) (layer B.Cu) (net 5))
@@
   (segment (start 161.399999 91.803999) (end 161.399999 89.806001) (width 0.65) (layer B.Cu) (net 35))
   (segment (start 162.179 92.583) (end 161.399999 91.803999) (width 0.65) (layer B.Cu) (net 35))
-  (segment (start 163.195 86.741) (end 163.195 84.963) (width 3) (layer F.Cu) (net 35))
   (segment (start 163.195 84.963) (end 163.195 85.979) (width 3) (layer F.Cu) (net 35))
   (segment (start 163.195 86.741) (end 164.465 86.741) (width 3) (layer F.Cu) (net 35))
@@
   (segment (start 161.720398 93.726) (end 161.769399 93.775001) (width 3) (layer F.Cu) (net 35))
   (segment (start 161.544 93.726) (end 161.720398 93.726) (width 3) (layer F.Cu) (net 35))
-  (segment (start 156.972 93.726) (end 161.544 93.726) (width 1) (layer F.Cu) (net 35))
   (segment (start 161.544 93.726) (end 163.195 93.726) (width 1) (layer F.Cu) (net 35))
   (segment (start 104.521 100.711) (end 111.379 107.569) (width 1) (layer F.Cu) (net 35))
@@
   (segment (start 97.343 85.151) (end 100.457 88.265) (width 0.5) (layer F.Cu) (net 35))
   (segment (start 97.343 81.595) (end 97.343 85.151) (width 0.5) (layer F.Cu) (net 35))
+  (segment (start 163.195 84.963) (end 168.275 84.963) (width 3) (layer F.Cu) (net 35))
+  (segment (start 168.275 84.963) (end 168.402 85.09) (width 3) (layer F.Cu) (net 35))
+  (segment (start 168.402 85.09) (end 168.402 86.614) (width 3) (layer F.Cu) (net 35))
+  (segment (start 167.259 87.757) (end 165.481 87.757) (width 3) (layer F.Cu) (net 35))
+  (segment (start 168.402 86.614) (end 167.259 87.757) (width 3) (layer F.Cu) (net 35))
+  (segment (start 161.544 93.726) (end 160.02 93.726) (width 3) (layer F.Cu) (net 35))
+  (segment (start 156.972 93.726) (end 160.02 93.726) (width 1) (layer F.Cu) (net 35))
+  (segment (start 163.195 86.741) (end 163.195 85.725) (width 3) (layer B.Cu) (net 35))
+  (segment (start 163.195 85.725) (end 163.576 85.344) (width 3) (layer B.Cu) (net 35))
+  (segment (start 163.576 85.344) (end 167.132 85.344) (width 3) (layer B.Cu) (net 35))
+  (segment (start 167.132 85.344) (end 168.148 86.36) (width 3) (layer B.Cu) (net 35))
+  (segment (start 168.148 86.36) (end 168.148 86.868) (width 3) (layer B.Cu) (net 35))
+  (segment (start 168.148 86.868) (end 167.181001 87.834999) (width 3) (layer B.Cu) (net 35))
+  (segment (start 167.181001 87.834999) (end 161.769399 87.834999) (width 3) (layer B.Cu) (net 35))
+  (segment (start 161.769399 87.834999) (end 160.224999 89.379399) (width 3) (layer B.Cu) (net 35))
+  (segment (start 160.224999 89.379399) (end 160.224999 92.406999) (width 3) (layer B.Cu) (net 35))
+  (segment (start 160.224999 92.406999) (end 161.798 93.98) (width 3) (layer B.Cu) (net 35))
+  (segment (start 161.798 93.98) (end 164.592 93.98) (width 3) (layer B.Cu) (net 35))
+  (segment (start 164.592 93.98) (end 166.37 92.202) (width 3) (layer B.Cu) (net 35))
+  (segment (start 166.37 92.202) (end 166.37 90.932) (width 3) (layer B.Cu) (net 35))
   (segment (start 72.6585 105.911) (end 72.517 105.7695) (width 0.65) (layer F.Cu) (net 36))
   (segment (start 75.547 105.911) (end 72.6585 105.911) (width 0.65) (layer F.Cu) (net 36))
@@
     )
   )
-  (zone (net 35) (net_name V_MMIC) (layer F.Cu) (hatch edge 0.508)
-    (connect_pads (clearance 0.6))
-    (min_thickness 0.254)
-    (fill yes (arc_segments 32) (thermal_gap 0.508) (thermal_bridge_width 0.508))
-    (polygon
-      (pts
-        (xy 188.341 100.203) (xy 188.341 112.141) (xy 116.713 112.141) (xy 116.713 100.203)
-      )
-    )
-  )
-  (zone (net 35) (net_name V_MMIC) (layer B.Cu) (hatch edge 0.508)
-    (connect_pads (clearance 0.508))
-    (min_thickness 0.254)
-    (fill yes (arc_segments 32) (thermal_gap 0.508) (thermal_bridge_width 0.508))
-    (polygon
-      (pts
-        (xy 169.037 82.677) (xy 169.037 95.885) (xy 159.385 95.885) (xy 159.385 82.677)
-      )
-    )
-  )
-  (zone (net 35) (net_name V_MMIC) (layer F.Cu) (hatch edge 0.508)
+  (zone (net 4) (net_name GND) (layer F.Cu) (hatch edge 0.508)
     (connect_pads (clearance 0.7))
     (min_thickness 0.254)
@@
     (polygon
       (pts
-        (xy 170.053 83.185) (xy 170.053 95.885) (xy 159.131 95.885) (xy 159.131 83.185)
+        (xy 208.788 128.27) (xy 66.04 128.27) (xy 66.04 41.148) (xy 208.788 41.148)
       )
     )
